File: proyecto.sch (EAGLE design)
At the start: 42 parts, among them IC1 ADE9153AACPZ, J1 796638-3, K1 PR28-3V-360-1A-E, Q1 12.288M, Q2 BSS123, U1 ESP32-PICO-MINI-02-N8R2ESP32-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

Commit message: MINI avance
No se avanzó tanto debido a que se me daño las pistas en plena clase :(
Connections:
- net CARGA: now also R3.4
Changed lines of the file:
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@@
 <label x="490.22" y="147.32" size="1.778" layer="95"/>
+</segment>
+<segment>
+<pinref part="R3" gate="G$1" pin="4"/>
+<wire x1="354.33" y1="99.06" x2="354.33" y2="100.33" width="0.1524" layer="91"/>
+<label x="354.33" y="98.806" size="1.778" layer="95" rot="R90"/>
 </segment>
 </net>

Commit message: Se añado y arreglo pistas
Se arreglo las pistas de la fase y el neutro en las clavijas. Se añadieron otras pistas y se quito el boton del enable.
Parts:
- removed S1: (no value), switch-omron:10-XX
- C1, C10, C11, C12, C13, C14, C15, C16, C17, C18, C19, C2, C20, C21, C22, C23, C3, C4, C5, C6, C7, C8, C9: device rcl:C-EUC0201 -> rcl:C-EUC0402K
- R9: device rcl:R-US_R1206 -> rcl:R-US_R0402
Connections:
- removed net N$14: C23.1, R9.2, S1.S
- net +3V3: now also R9.1
- net CF1: now also U1.IO12
- net EN: now also C23.1, R9.2; no longer R9.1
- net GND: now also U1.GND, U1.GND_10, U1.GND_11, U1.GND_12, U1.GND_13, U1.GND_14, U1.GND_15, U1.GND_16, U1.GND_17, U1.GND_18, U1.GND_19, U1.GND_2, U1.GND_20, U1.GND_21, U1.GND_22, U1.GND_23, U1.GND_24, U1.GND_25, U1.GND_26, U1.GND_27, U1.GND_28, U1.GND_29, U1.GND_3, U1.GND_30, U1.GND_4, U1.GND_5, U1.GND_6, U1.GND_7, U1.GND_8, U1.GND_9; no longer S1.P
- net IRQ: now also U1.IO14
- net NEUTRO: now also R4.1
- net RELAY_CONTROL: now also U1.IO13
- net RESET: now also U1.IO27
- net RX: now also U1.IO26
- net SCLK: now also U1.IO33; no longer U1.I37
- net SS: now also U1.IO32; no longer U1.I36
- net TX: now also U1.IO25
Other:
- moved on the sheet: C23, R9

Commit message: Terminada la mayoria de conexiones
Se realizo la gran mayoria de las conexiones, falta realizar las conexiones especificadas en el DRC.
Parts:
- added S1: 3-1437565-0, SamacSys_Parts:3-1437565-0
- R1, R2: device rcl:R-US_R0201 -> rcl:R-US_R0402
- SV1: device con-lstb:MA04-1 -> con-lsta:FE06-1
Connections:
- net CARGA_M renamed MONDA
- net N$11 renamed PROG_TX
- net N$12 renamed PROG_RX
- removed net VDD1: C1.1, C2.1, IC1.VDD_1
- removed net VDD2: C3.1, C4.1, IC1.VDD_2
- new net BOOT: S1.COM_1, S1.COM_2, SV1.4, U1.IO0
- net +3V3: now also C1.1, C2.1, C3.1, C4.1, IC1.VDD_1, IC1.VDD_2
- net EN: now also SV1.5
- net GND: now also S1.NO_1, S1.NO_2, SV1.6; no longer SV1.4
