File: proyecto.brd (EAGLE design)
At the start: 95.8 x 48.2 mm, 51 parts, among them IC1 ADE9153AACPZ, J1 796638-3, K1 PR28-3V-360-1A-E, Q1 12.288M, Q2 BSS123, U1 ESP32-PICO-MINI-02-N8R2ESP32-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

Commit message: .
.
Parts:
- moved TP3 21.0 mm to (-9.53, -20.0), flipped to the bottom
- moved TP1 7.77 mm to (19.9, 4.11), flipped to the bottom
- moved SV1 3.96 mm to (26.3, 21.7)
- flipped TP4 to the bottom
Connections:
- net CARGA renamed M
Routing:
- net GND: track 27.1 -> 34.8 mm
- net RELAY_CONTROL: track 25.2 -> 32.4 mm, vias 0 -> 1
- net LINEA: track 67.3 -> 72.1 mm
- net M: track 0.00 -> 4.39 mm, vias 8 -> 15
- net EN: track 33.7 -> 37.7 mm
- net PROG_RX: track 9.94 -> 13.9 mm
- net PROG_TX: track 7.11 -> 11.1 mm
- net BOOT: track 23.0 -> 27.0 mm
- net +3V3: track 136.1 -> 137.9 mm, vias 7 -> 5
- net RELAY: track 15.6 -> 15.8 mm, vias 1 -> 0

Commit message: Supongo que ya es el final
:)
Parts:
- moved TP3 2.81 mm to (-6.71, -20.0)
Routing:
- net +3V3: track 137.9 -> 137.3 mm
- net GND: track 34.8 -> 34.4 mm, vias 19 -> 45
- added copper zone on layer 1, net +3V3
- removed copper zone on layer 16, net RELAY

Commit message: todo listo
:)
Routing:
- net GND: track 34.4 -> 31.8 mm
Changed lines of the file:
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@@
 <vertex x="25.5778" y="-7.62"/>
 <vertex x="21.6916" y="-3.7338"/>
-<vertex x="25.5778" y="-7.62"/>
 </polygon>
 <polygon width="2" layer="30">
@@
 <wire x1="6.58" y1="17.7135" x2="6.63" y2="17.6635" width="0.3" layer="1"/>
 <wire x1="7.43" y1="17.6635" x2="8.23" y2="17.6635" width="0.3" layer="1"/>
-<wire x1="5.48" y1="17.7135" x2="5.0893" y2="17.3228" width="0.3" layer="1"/>
-<wire x1="5.0893" y1="17.3228" x2="4.4958" y2="17.3228" width="0.3" layer="1"/>
 <wire x1="17.38" y1="17.7135" x2="16.28" y2="17.7135" width="0.3" layer="1"/>
 <wire x1="16.28" y1="17.7135" x2="16.23" y2="17.6635" width="0.3" layer="1"/>
 <wire x1="16.23" y1="17.6635" x2="15.43" y2="17.6635" width="0.3" layer="1"/>
-<wire x1="17.38" y1="17.7135" x2="18.0751" y2="17.7135" width="0.3" layer="1"/>
-<wire x1="18.0751" y1="17.7135" x2="18.5928" y2="17.1958" width="0.3" layer="1"/>
 <via x="19.023328125" y="-9.9822" extent="1-16" drill="0.35"/>
 <via x="20.293328125" y="-9.9822" extent="1-16" drill="0.35"/>
@@
 <via x="-22.7876125" y="-8.898890625" extent="1-16" drill="0.35"/>
 <via x="-21.5176125" y="-8.898890625" extent="1-16" drill="0.35"/>
+<polygon width="0.1524" layer="1" thermals="no">
+<vertex x="5.24636875" y="17.865090625"/>
+<vertex x="4.949190625" y="17.865090625"/>
+<vertex x="4.606290625" y="17.522190625"/>
+<vertex x="4.606290625" y="17.2593"/>
+<vertex x="4.81203125" y="17.053559375"/>
+<vertex x="4.81203125" y="17.236440625"/>
+<vertex x="5.15493125" y="17.579340625"/>
+<vertex x="5.234940625" y="17.579340625"/>
+<vertex x="5.234940625" y="17.8536625"/>
+</polygon>
+<polygon width="0.1524" layer="1" thermals="no">
+<vertex x="17.693640625" y="17.88795"/>
+<vertex x="18.585178125" y="17.88795"/>
+<vertex x="18.73376875" y="17.739359375"/>
+<vertex x="18.73376875" y="17.68220625"/>
+<vertex x="18.35658125" y="17.30501875"/>
+<vertex x="18.219421875" y="17.30501875"/>
+<vertex x="17.910809375" y="17.61363125"/>
+<vertex x="17.682209375" y="17.61363125"/>
+<vertex x="17.682209375" y="17.88795"/>
+</polygon>
 </signal>
 <signal name="AVDDOUT">
@@
 <vertex x="35.5854" y="-0.508"/>
 </polygon>
-<wire x1="20.2438" y1="-2.2606" x2="25.6032" y2="-7.62" width="3" layer="16"/>
+<wire x1="20.2438" y1="-2.2606" x2="22.056090625" y2="-4.072890625" width="3" layer="16"/>
+<wire x1="25.6032" y1="-7.62" x2="22.056090625" y2="-4.072890625" width="3" layer="16"/>
 <wire x1="25.6032" y1="-7.62" x2="29.8958" y2="-7.62" width="3" layer="16"/>
 <wire x1="37.1348" y1="-0.381" x2="37.1348" y2="3.1242" width="3" layer="16"/>
@@
 <via x="42.3164" y="1.0668" extent="1-16" drill="0.35"/>
 <via x="44.323" y="1.0922" extent="1-16" drill="0.35"/>
-<wire x1="17.8562" y1="-4.6482" x2="21.1836" y2="-4.6482" width="0.8" layer="16"/>
-<wire x1="22.0472" y1="-5.5118" x2="22.5806" y2="-5.5118" width="0.8" layer="16"/>
-<wire x1="21.1836" y1="-4.6482" x2="22.0472" y2="-5.5118" width="0.8" layer="16"/>
 <via x="43.3578" y="1.0922" extent="1-16" drill="0.35"/>
+<wire x1="22.056090625" y1="-4.072890625" x2="22.056090625" y2="-4.072890625" width="3" layer="16"/>
+<wire x1="22.056090625" y1="-4.072890625" x2="21.625559375" y2="-4.503421875" width="1" layer="16"/>
+<wire x1="21.625559375" y1="-4.503421875" x2="21.625559375" y2="-4.98348125" width="1" layer="16"/>
+<wire x1="21.625559375" y1="-4.98348125" x2="19.3167" y2="-4.98348125" width="1" layer="16"/>
+<wire x1="19.3167" y1="-4.98348125" x2="19.3167" y2="-4.4577" width="1" layer="16"/>
+<wire x1="19.3167" y1="-4.4577" x2="19.579590625" y2="-4.194809375" width="1" layer="16"/>
+<wire x1="19.579590625" y1="-4.194809375" x2="20.24253125" y2="-4.194809375" width="1" layer="16"/>
 </signal>
 <signal name="TIERRA">
@@
 <mfgpreviewcolor name="substratecolor" color="0xFF786E46"/>
 </mfgpreviewcolors>
-<errors>
-</errors>
 </board>
 </drawing>

Commit message: XDIN
XDIN
Parts:
- removed Q1: 12.288M, crystal-geyer_V1_0:2.0X1.6_KX-5
- added Y1: NX3225GA-12.288M-STD-CRG-2, SamacSys_Parts:NX3225GA12288MSTDCRG2
Connections:
- net CLKIN: now also Y1.1; no longer Q1.1
- net CLKOUT: now also Y1.3; no longer Q1.3
- net GND: now also Y1.2, Y1.4
Routing:
- net GND: track 31.8 -> 35.8 mm, vias 45 -> 46
- net CLKIN: track 13.8 -> 14.6 mm
- net +3V3: track 137.3 -> 136.6 mm
